File: monitor_system.kicad_sch (KiCad schematic)
At the start: 16 parts, among them K1 DIPxx-1Axx-11x, Q1 2N7002, U1 NE555D, U2 L7805, U3 LM393, U4 7400, U5 ACS780xLRTR-050U

Commit message: feat + fix + refactor on kicad pcb
feat:added components connections

fix: fixed DRC clearence errors

refactor:moved components in a different layout

ERC: passed warnings(3)
DRC: passed no warnings
Parts:
- U3: footprint (none) -> Package_DIP:DIP-8-16_W7.62mm
- U4: footprint (none) -> Package_DIP:DIP-14_W7.62mm
Changed lines of the file:
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@@
 			)
 		)
-		(property "Footprint" ""
+		(property "Footprint" "Package_DIP:DIP-14_W7.62mm"
 			(at 219.71 127 0)
 			(effects
@@
 			)
 		)
-		(property "Footprint" ""
+		(property "Footprint" "Package_DIP:DIP-14_W7.62mm"
 			(at 57.15 138.43 0)
 			(effects
@@
 			)
 		)
-		(property "Footprint" ""
+		(property "Footprint" "Package_DIP:DIP-14_W7.62mm"
 			(at 57.15 125.73 0)
 			(effects
@@
 			)
 		)
-		(property "Footprint" ""
+		(property "Footprint" "Package_DIP:DIP-8-16_W7.62mm"
 			(at 123.19 134.62 0)
 			(effects
@@
 			)
 		)
-		(property "Footprint" ""
+		(property "Footprint" "Package_DIP:DIP-8-16_W7.62mm"
 			(at 233.68 123.19 0)
 			(effects
@@
 			)
 		)
-		(property "Footprint" ""
+		(property "Footprint" "Package_DIP:DIP-14_W7.62mm"
 			(at 82.55 140.97 0)
 			(effects
@@
 			)
 		)
-		(property "Footprint" ""
+		(property "Footprint" "Package_DIP:DIP-14_W7.62mm"
 			(at 82.55 124.46 0)
 			(effects
